File: OVEN_SWITCH.kicad_pcb (KiCad board)
At the start: 2 copper layers, 366 x 97.5 mm, 32 parts, among them J1 CONN_01X17, SW10 BAKED GOODS, SW11 MEATS, SW12 OTHER FOODS, SW13 COOK TIME, SW14 STOP TIME, SW15 CONVECT FULL MEAL, SW16 7, SW17 4, SW18 1, SW19 0, SW2 LOWER OVEN, SW20 8, SW21 5, SW22 2, SW23 6, SW24 OVEN LIGHT, SW25 9, SW26 3, SW27 SET.START, SW28 CLOCK, SW29 CANCEL, SW3 UPPER OVEN, SW30 LOWER OVEN CANCEL/OFF, SW31 UPPER OVEN CANCEL/OFF, SW32 START, SW4 BAKE, SW5 BAKE, SW6 BROIL, SW7 BROIL, SW8 CLEAN, SW9 ROAST

Commit message: Add files via upload
before moving edge and connector
Parts:
- moved SW28 135.3 mm to (189.1, 126.6)
- moved SW10 135.3 mm to (1.56, 129.1)
- moved SW11 135.3 mm to (21.6, 129.1)
- moved SW12 135.3 mm to (41.6, 129.1)
- moved SW13 135.3 mm to (71.6, 121.6)
- moved SW14 135.3 mm to (71.6, 136.6)
- moved SW2 135.3 mm to (-98.4, 136.6)
- moved SW3 135.3 mm to (-98.4, 121.6)
- moved SW4 135.3 mm to (-68.4, 136.6)
- moved SW5 135.3 mm to (-68.4, 121.6)
- moved J1 135.3 mm to (130.3, 63.9)
- moved SW19 135.1 mm to (121.6, 135.1)
- moved SW20 135.1 mm to (121.6, 117.6)
- moved SW21 135.1 mm to (121.6, 100.1)
- moved SW22 135.1 mm to (121.6, 82.6)
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Routing:
- net Net-(J1-Pad9): track 425.0 -> 777.9 mm, vias 6 -> 5
- net Net-(J1-Pad14): track 243.5 -> 494.2 mm, vias 12 -> 11
- net Net-(J1-Pad7): track 474.7 -> 545.4 mm, vias 10 -> 13
- net Net-(J1-Pad15): track 547.8 -> 576.0 mm, vias 8 -> 12
- net Net-(J1-Pad12): track 146.3 -> 121.8 mm, vias 8 -> 6
- net Net-(J1-Pad2): track 462.7 -> 446.2 mm, vias 3 -> 2
- net Net-(J1-Pad11): track 116.2 -> 124.3 mm
- net Net-(J1-Pad13): track 112.5 -> 108.0 mm
- net Net-(J1-Pad10): track 143.9 -> 146.6 mm, vias 6 -> 4
- net Net-(J1-Pad4): track 495.1 -> 492.6 mm, vias 10 -> 8
- net Net-(J1-Pad3): track 359.0 -> 359.1 mm, vias 11 -> 7
Other:
- outline, holes or cut-outs redrawn

Commit message: Add files via upload
files after first CNC prototype of left half
Parts:
- removed the SW28 at (189.1, 126.6)
- added SW27: CLOCK, data:Membrane_Switch_Wide, F.Cu at (332.2, 124.3)
- moved J1 160.3 mm to (290.6, 66.8)
- moved SW13 152.1 mm to (223.7, 137.3)
- moved SW11 152.1 mm to (193.7, 128.8)
- moved SW12 152.1 mm to (223.7, 121.3)
- moved SW14 152.1 mm to (253.7, 134.8)
- moved SW15 152.1 mm to (253.7, 117.3)
- moved SW18 152.1 mm to (273.7, 134.8)
- moved SW19 152.1 mm to (273.7, 117.3)
- moved SW20 152.1 mm to (273.7, 99.8)
- moved SW21 152.1 mm to (273.7, 82.3)
- moved SW22 152.1 mm to (293.7, 99.8)
- moved SW23 152.1 mm to (293.7, 134.8)
- moved SW24 152.1 mm to (293.7, 117.3)
- moved SW25 152.1 mm to (293.7, 82.3)
- moved SW16 152.1 mm to (253.6, 99.9)
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- renumbered SW2 to SW1, SW11 to SW10, SW12 to SW11, SW13 to SW12, SW14 to SW13, SW15 to SW14, SW16 to SW15, SW17 to SW16, SW18 to SW17, SW19 to SW18, SW20 to SW19, SW3 to SW2, SW21 to SW20, SW22 to SW21, SW23 to SW22, SW24 to SW23, SW25 to SW24, SW26 to SW25, SW27 to SW26, SW29 to SW28, SW30 to SW29, SW4 to SW3, SW31 to SW30, SW32 to SW31, SW5 to SW4, SW6 to SW5, SW7 to SW6, SW8 to SW7, SW9 to SW8, SW10 to SW9
Routing:
- net Net-(J1-Pad9): track 777.9 -> 553.5 mm, vias 5 -> 4
- net Net-(J1-Pad14): track 494.2 -> 273.8 mm, vias 11 -> 4
- net Net-(J1-Pad2): track 446.2 -> 515.6 mm, vias 2 -> 14
- net Net-(J1-Pad3): track 359.1 -> 404.9 mm, vias 7 -> 24
- net Net-(J1-Pad4): track 492.6 -> 532.7 mm, vias 8 -> 9
- net Net-(J1-Pad13): track 108.0 -> 130.7 mm, vias 4 -> 2
- net Net-(J1-Pad10): track 146.6 -> 125.1 mm, vias 4 -> 2
- net Net-(J1-Pad12): track 121.8 -> 141.8 mm, vias 6 -> 4
- net Net-(J1-Pad15): track 576.0 -> 556.0 mm, vias 12 -> 10
- net Net-(J1-Pad7): track 545.4 -> 530.4 mm, vias 13 -> 14
- net Net-(J1-Pad1): track 49.6 -> 42.0 mm, vias 1 -> 0
- net Net-(J1-Pad11): track 124.3 -> 124.7 mm, vias 6 -> 2
Other:
- board size 366 x 97.5 mm -> 366 x 89.5 mm
- net class Default: trace_width 0.5 -> 1
